Commit message: Working Version

File: urdf/ur5e_sc_down.urdf (robot description, URDF)
Before this commit: robot ur5e, 13 links, 12 joints
Links:
- link suction_cylinder: geometry collision cylinder length=0.15 radius=0.02; visual cylinder length=0.15 radius=0.02
Joints:
- joint ee_fixed_joint: origin xyz=0.0 0.1 0.0 rpy=-1.57079632679 0 0 -> xyz=0.0 0.1 0.0 rpy=-1.57079632679 0.0 0.0
- joint elbow_joint: limit lower=-3.14159265359 upper=3.14159265359 effort=150.0 velocity=3.14 -> lower=-9.14159265359 upper=9.14159265359 effort=150.0 velocity=3.14; origin xyz=0.0 -0.131 0.425 rpy=0.0 0.0 0.0 -> xyz=0.0 -0.131 0.425 rpy=0.0 -2.35619449019 0.0
- joint shoulder_lift_joint: limit lower=-6.28318530718 upper=6.28318530718 effort=150.0 velocity=3.14 -> lower=-9.28318530718 upper=9.28318530718 effort=150.0 velocity=3.14
- joint suction_joint: origin xyz=0 0 0.025 rpy=0 0 0 -> xyz=0 0 0.075 rpy=0 0 0
- joint suction_tip_joint: origin xyz=0 0 0.025 rpy=0 0 0 -> xyz=0 0 0.075 rpy=0 3.14159 0
- joint world_joint: origin xyz=0.0 0.0 0.0 rpy=0.0 0.0 0.0 -> xyz=0.0 0.0 0.0 rpy=3.14159265359 0.0 0.0
- joint wrist_1_joint: limit lower=-6.28318530718 upper=6.28318530718 effort=28.0 velocity=6.28 -> lower=-9.28318530718 upper=9.28318530718 effort=28.0 velocity=6.28; origin xyz=0.0 0.0 0.392 rpy=0.0 1.57079632679 0.0 -> xyz=0.0 0.0 0.392 rpy=0.0 0.0 0.0
- joint wrist_2_joint: limit lower=-6.28318530718 upper=6.28318530718 effort=28.0 velocity=6.28 -> lower=-9.28318530718 upper=9.28318530718 effort=28.0 velocity=6.28; origin xyz=0.0 0.127 0.0 rpy=0.0 0.0 0.0 -> xyz=0.0 0.127 0.0 rpy=0.0 0.0 -1.57079632679
- joint wrist_3_joint: limit lower=-6.28318530718 upper=6.28318530718 effort=28.0 velocity=6.28 -> lower=-9.28318530718 upper=9.28318530718 effort=28.0 velocity=6.28
- joint wrist_3_link-tool0_fixed_joint: origin xyz=0 0.1 0 rpy=-1.57079632679 0 -1.57079632679 -> xyz=0 0.1 0 rpy=-1.57079632679 0 0
